File: Tirusse_hw/Tirusse.kicad_sch (KiCad schematic)
At the start: 237 parts

Commit message: + Radio works + Blade powered off and on * SCH modified to fix powerbtn control
Connections:
- net +BAT_IN is gone; now on net +BATT: U.1, U.1, U.1 (P1), U.1 (P1), U.2, U.2, U.2, U.2 (S), U.2 (S), U.5 (BAT), U.C
- net PWRBTN1 is gone; now on net ACC_INT1: U.1, U.1, U.1 (G)
Other:
- note added: "10k"
- note added: "Always on"
- note added: "Do not mount"
- note added: "Power on"
